Commit message: update sample codes

File: ir_gazebo/urdf/table.urdf.xacro (robot description, xacro)
@@ -5,10 +5,10 @@
     <visual>
        <geometry>
-	   <box size="0.07 0.07 0.7"/>
+	   <box size="0.07 0.07 0.735"/>
 	</geometry>
     </visual>
     <collision>
        <geometry>
-	   <box size="0.07 0.07 0.7"/>
+	   <box size="0.07 0.07 0.735"/>
 	</geometry>
     </collision>
@@ -33,10 +33,10 @@
     <visual>
        <geometry>
-	   <box size="0.9 1.7 0.05"/>
+	   <box size="0.9 1.2 0.05"/>
 	</geometry>
     </visual>
     <collision>
        <geometry>
-	   <box size="0.9 1.7 0.05"/>
+	   <box size="0.9 1.2 0.05"/>
 	</geometry>
     </collision>
@@ -56,5 +56,5 @@
     <parent link="column"/>
     <child link="surface"/>
-    <origin xyz ="0 0 0.375" rpy= "0 0 0"/> <!--z axis: {height}/2 -->
+    <origin xyz ="0 0 0.3925" rpy= "0 0 0"/> <!--z axis: {height}/2 -->
   </joint>
 </robot>

File: ir_gazebo/urdf/ur5e_rg2.urdf.xacro (robot description, xacro)
@@ -26,10 +26,10 @@
     <parent link="workstation_link" />
     <child link = "base_link" />
-    <origin xyz="0.0 0.0 0.375" rpy="0.0 0.0 0.0" />
+    <origin xyz="0.18 0.0 0.395" rpy="0.0 0.0 0.0" />
   </joint>
   <joint name="world_joint" type="fixed">
     <parent link="world" />
     <child link = "table_base_link" />
-    <origin xyz="0.8 0.0 0.0" rpy="0.0 0.0 0.0" />
+    <origin xyz="1.2 0.0 0.0" rpy="0.0 0.0 0.0" />
   </joint>
   <gazebo>

File: ir_gazebo/urdf/workstation.urdf.xacro (robot description, xacro)
@@ -7,12 +7,12 @@
     <visual>
       <geometry>
-	      <box size="0.3 1.5 0.75"/>
+	      <box size="0.76 0.72 0.79"/>
 	    </geometry>
-      <material name="white"/>
+      <material name="white_workstation"/>
     </visual>
     <collision>
-       <geometry>
-	   <box size="0.3 1.5 0.75"/>
-	</geometry>
+      <geometry>
+	      <box size="0.76 0.72 0.79"/>
+	    </geometry>
     </collision>
     <inertial>
@@ -32,5 +32,5 @@
     <parent link="world" />
     <child link = "workstation_link" />
-    <origin xyz="0. 0. 0.375" rpy="0.0 0.0 0.0" />
+    <origin xyz="0. 0. 0.395" rpy="0.0 0.0 0.0" />
   </joint>
 </robot>
