Commit message: update demo codes

File: ir_gazebo/urdf/ur5e_rg2.urdf.xacro (robot description, xacro)
@@ -31,5 +31,5 @@
     <parent link="world" />
     <child link = "table_base_link" />
-    <origin xyz="1.2 0.0 0.0" rpy="0.0 0.0 0.0" />
+    <origin xyz="0.83 0.0 0.0" rpy="0.0 0.0 0.0" /> <!--0.76/2+0.9/2-->
   </joint>
   <gazebo>
