Commit message: update realsense dependency

File: ir_gazebo/urdf/realsense_d435/d435.urdf.xacro (robot description, xacro)
@@ -48,6 +48,5 @@
         <geometry>
           <!-- <box size="${d435_cam_width} ${d435_cam_height} ${d435_cam_depth}"/> -->
-          <mesh filename="package://realsense2_description/meshes/d435.dae" />
-          <!--<mesh filename="package://realsense2_description/meshes/d435/d435.dae" />-->
+          <mesh filename="package://ir_gazebo/urdf/realsense_d435/meshes/visual/d435.dae" />
         </geometry>
         <material name="${name}_aluminum"/>
