Commit message: update tcp joint

File: ir_gazebo/script/structure/utils/ur5e_onrobot.urdf (robot description, URDF)
Before this commit: robot rilab_robot, 15 links, 14 joints
Links:
- added link gripper_tcp_link, mass 0.199035856566616
Joints:
- added joint gripper_tcp_joint: type fixed, parent gripper_base_link, child gripper_tcp_link, origin xyz=-0.00725 0.11 0. rpy=0 0 0, axis 0 0 0
- joint gripper_base_joint: origin xyz=0 0 0 rpy=-1.57 0 0 -> xyz=0 0. 0. rpy=0 0 0

Commit message: clean code

File: ir_gazebo/script/structure/utils/ur5e_onrobot.urdf (robot description, URDF)
Before this commit: robot rilab_robot, 16 links, 15 joints
Joints:
- joint gripper_tcp_joint: axis 0 0 0 -> 0 1 0; origin xyz=-0.00725 0.11 0. rpy=0 0 0 -> xyz=0 0.16 0 rpy=0 0 0
